File: BSB-LAN-Full-Wifi.sch (EAGLE design)
At the start: 70 parts, among them IC4 SY8089AAAC, IC6 CH340X, Q1 BC847, Q2 BC857, Q5 BC847, Q6 BC847, Q7 WPM2015-3/TR, U2 ESDS314DBV

Commit message: Add Missing LCSC_PART Attributes on BSB-LAN-Full-Wifi
Missing TVS and DC-DC JLC assembly part numbers.
Parts:
- D1: LCSC_PART (none) -> C148213
Changed lines of the file:
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@@
 <grid distance="0.1" unitdist="inch" unit="inch" style="lines" multiple="1" display="no" altdistance="0.01" altunitdist="inch" altunit="inch"/>
 <layers>
-<layer number="1" name="Top" color="4" fill="1" visible="yes" active="no"/>
-<layer number="2" name="Route2" color="1" fill="3" visible="yes" active="no"/>
-<layer number="3" name="Route3" color="4" fill="3" visible="yes" active="no"/>
-<layer number="4" name="Route4" color="1" fill="4" visible="yes" active="no"/>
-<layer number="5" name="Route5" color="4" fill="4" visible="yes" active="no"/>
-<layer number="6" name="Route6" color="1" fill="8" visible="yes" active="no"/>
-<layer number="7" name="Route7" color="4" fill="8" visible="yes" active="no"/>
-<layer number="8" name="Route8" color="1" fill="2" visible="yes" active="no"/>
-<layer number="9" name="Route9" color="4" fill="2" visible="yes" active="no"/>
-<layer number="10" name="Route10" color="1" fill="7" visible="yes" active="no"/>
-<layer number="11" name="Route11" color="4" fill="7" visible="yes" active="no"/>
-<layer number="12" name="Route12" color="1" fill="5" visible="yes" active="no"/>
-<layer number="13" name="Route13" color="4" fill="5" visible="yes" active="no"/>
-<layer number="14" name="Route14" color="1" fill="6" visible="yes" active="no"/>
-<layer number="15" name="Route15" color="4" fill="6" visible="yes" active="no"/>
-<layer number="16" name="Bottom" color="1" fill="1" visible="yes" active="no"/>
-<layer number="17" name="Pads" color="2" fill="1" visible="yes" active="no"/>
-<layer number="18" name="Vias" color="2" fill="1" visible="yes" active="no"/>
-<layer number="19" name="Unrouted" color="6" fill="1" visible="yes" active="no"/>
-<layer number="20" name="Dimension" color="15" fill="1" visible="yes" active="no"/>
-<layer number="21" name="tPlace" color="7" fill="1" visible="yes" active="no"/>
-<layer number="22" name="bPlace" color="7" fill="1" visible="yes" active="no"/>
-<layer number="23" name="tOrigins" color="15" fill="1" visible="yes" active="no"/>
-<layer number="24" name="bOrigins" color="15" fill="1" visible="yes" active="no"/>
-<layer number="25" name="tNames" color="7" fill="1" visible="yes" active="no"/>
-<layer number="26" name="bNames" color="7" fill="1" visible="yes" active="no"/>
-<layer number="27" name="tValues" color="7" fill="1" visible="yes" active="no"/>
-<layer number="28" name="bValues" color="7" fill="1" visible="yes" active="no"/>
+<layer number="1" name="Top" color="4" fill="1" visible="no" active="no"/>
+<layer number="2" name="Route2" color="1" fill="3" visible="no" active="no"/>
+<layer number="3" name="Route3" color="4" fill="3" visible="no" active="no"/>
+<layer number="4" name="Route4" color="1" fill="4" visible="no" active="no"/>
+<layer number="5" name="Route5" color="4" fill="4" visible="no" active="no"/>
+<layer number="6" name="Route6" color="1" fill="8" visible="no" active="no"/>
+<layer number="7" name="Route7" color="4" fill="8" visible="no" active="no"/>
+<layer number="8" name="Route8" color="1" fill="2" visible="no" active="no"/>
+<layer number="9" name="Route9" color="4" fill="2" visible="no" active="no"/>
+<layer number="10" name="Route10" color="1" fill="7" visible="no" active="no"/>
+<layer number="11" name="Route11" color="4" fill="7" visible="no" active="no"/>
+<layer number="12" name="Route12" color="1" fill="5" visible="no" active="no"/>
+<layer number="13" name="Route13" color="4" fill="5" visible="no" active="no"/>
+<layer number="14" name="Route14" color="1" fill="6" visible="no" active="no"/>
+<layer number="15" name="Route15" color="4" fill="6" visible="no" active="no"/>
+<layer number="16" name="Bottom" color="1" fill="1" visible="no" active="no"/>
+<layer number="17" name="Pads" color="2" fill="1" visible="no" active="no"/>
+<layer number="18" name="Vias" color="2" fill="1" visible="no" active="no"/>
+<layer number="19" name="Unrouted" color="6" fill="1" visible="no" active="no"/>
+<layer number="20" name="Dimension" color="15" fill="1" visible="no" active="no"/>
+<layer number="21" name="tPlace" color="7" fill="1" visible="no" active="no"/>
+<layer number="22" name="bPlace" color="7" fill="1" visible="no" active="no"/>
+<layer number="23" name="tOrigins" color="15" fill="1" visible="no" active="no"/>
+<layer number="24" name="bOrigins" color="15" fill="1" visible="no" active="no"/>
+<layer number="25" name="tNames" color="7" fill="1" visible="no" active="no"/>
+<layer number="26" name="bNames" color="7" fill="1" visible="no" active="no"/>
+<layer number="27" name="tValues" color="7" fill="1" visible="no" active="no"/>
+<layer number="28" name="bValues" color="7" fill="1" visible="no" active="no"/>
 <layer number="29" name="tStop" color="7" fill="3" visible="no" active="no"/>
 <layer number="30" name="bStop" color="7" fill="6" visible="no" active="no"/>
@@
 <layer number="35" name="tGlue" color="7" fill="4" visible="no" active="no"/>
 <layer number="36" name="bGlue" color="7" fill="5" visible="no" active="no"/>
-<layer number="37" name="tTest" color="7" fill="1" visible="yes" active="no"/>
-<layer number="38" name="bTest" color="7" fill="1" visible="yes" active="no"/>
+<layer number="37" name="tTest" color="7" fill="1" visible="no" active="no"/>
+<layer number="38" name="bTest" color="7" fill="1" visible="no" active="no"/>
 <layer number="39" name="tKeepout" color="4" fill="11" visible="no" active="no"/>
 <layer number="40" name="bKeepout" color="1" fill="11" visible="no" active="no"/>
@@
 <layer number="44" name="Drills" color="7" fill="1" visible="no" active="no"/>
 <layer number="45" name="Holes" color="7" fill="1" visible="no" active="no"/>
-<layer number="46" name="Milling" color="3" fill="1" visible="yes" active="no"/>
-<layer number="47" name="Measures" color="7" fill="1" visible="yes" active="no"/>
-<layer number="48" name="Document" color="7" fill="1" visible="yes" active="no"/>
-<layer number="49" name="Reference" color="7" fill="1" visible="yes" active="no"/>
-<layer number="50" name="dxf" color="7" fill="1" visible="yes" active="no"/>
-<layer number="51" name="tDocu" color="7" fill="1" visible="yes" active="no"/>
-<layer number="52" name="bDocu" color="7" fill="1" visible="yes" active="no"/>
-<layer number="53" name="tGND_GNDA" color="7" fill="9" visible="yes" active="no"/>
-<layer number="54" name="bGND_GNDA" color="1" fill="9" visible="yes" active="no"/>
-<layer number="56" name="wert" color="7" fill="1" visible="yes" active="no"/>
-<layer number="57" name="tCAD" color="7" fill="1" visible="yes" active="no"/>
-<layer number="58" name="bCAD" color="7" fill="1" visible="yes" active="no"/>
-<layer number="59" name="tCarbon" color="7" fill="1" visible="yes" active="no"/>
-<layer number="60" name="bCarbon" color="7" fill="1" visible="yes" active="no"/>
+<layer number="46" name="Milling" color="3" fill="1" visible="no" active="no"/>
+<layer number="47" name="Measures" color="7" fill="1" visible="no" active="no"/>
+<layer number="48" name="Document" color="7" fill="1" visible="no" active="no"/>
+<layer number="49" name="Reference" color="7" fill="1" visible="no" active="no"/>
+<layer number="50" name="dxf" color="7" fill="1" visible="no" active="no"/>
+<layer number="51" name="tDocu" color="7" fill="1" visible="no" active="no"/>
+<layer number="52" name="bDocu" color="7" fill="1" visible="no" active="no"/>
+<layer number="53" name="tGND_GNDA" color="7" fill="9" visible="no" active="no"/>
+<layer number="54" name="bGND_GNDA" color="1" fill="9" visible="no" active="no"/>
+<layer number="56" name="wert" color="7" fill="1" visible="no" active="no"/>
+<layer number="57" name="tCAD" color="7" fill="1" visible="no" active="no"/>
+<layer number="58" name="bCAD" color="7" fill="1" visible="no" active="no"/>
+<layer number="59" name="tCarbon" color="7" fill="1" visible="no" active="no"/>
+<layer number="60" name="bCarbon" color="7" fill="1" visible="no" active="no"/>
 <layer number="88" name="SimResults" color="9" fill="1" visible="yes" active="yes"/>
 <layer number="89" name="SimProbes" color="9" fill="1" visible="yes" active="yes"/>
@@
 </part>
 <part name="12V" library="BSB-LAN" deviceset="MKDSN1,5/2-5,08" device=""/>
-<part name="D1" library="BSB-LAN" deviceset="TVS-UNI" device="SMA" value="12V"/>
+<part name="D1" library="BSB-LAN" deviceset="TVS-UNI" device="SMA" value="12V">
+<attribute name="LCSC_PART" value="C148213"/>
+</part>
 </parts>
 <sheets>

Commit message: Reduce Wifi BoM Complexity
There were some weird values left that were holdovers from the LAN board where they were used elsewhere.
Parts:
- C18: value 220uF 25V -> 100uF 20V; LCSC_PART (none) -> C7224
- C20, C21: value 1nF 3kV -> 1nF 2kV; device BSB-LAN:C-EUC1808 -> BSB-LAN:C-EUC1206L; LCSC_PART C577300 -> C9196
- D6: value SS510B -> SS34; device BSB-LAN:DIODE-SMB -> BSB-LAN:DIODE-SMA; LCSC_PART C65011 -> C8678
- R40, R43: value 180k 1% -> 200k 1%; LCSC_PART C25760 -> C25764
- R41: value 12.1k 1% -> 22k 1%; LCSC_PART C25852 -> C25768
- R42: value 28.7k 1% -> 22k 1%; LCSC_PART C26972 -> C25768
Other:
- note added: "Vout = 0.6 x (200/44 + 1) = 3.32V"
- note removed: "Vout = 0.6 x (180/40.8 + 1) = 3.25V"
Changed lines of the file:
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@@
 </class>
 <class number="2" name="PoE-ISO" width="0" drill="0">
-<clearance class="1" value="2"/>
+<clearance class="1" value="1.7"/>
 </class>
 <class number="3" name="B2B-ISO" width="0" drill="0">
-<clearance class="1" value="2"/>
-<clearance class="2" value="2"/>
+<clearance class="1" value="1.7"/>
+<clearance class="2" value="1.7"/>
 </class>
 <class number="4" name="ESP32" width="0" drill="0">
-<clearance class="2" value="2"/>
-<clearance class="3" value="2"/>
+<clearance class="2" value="1.7"/>
+<clearance class="3" value="1.7"/>
 </class>
 <class number="5" name="Sheild" width="0" drill="0">
 <clearance class="1" value="1.5"/>
-<clearance class="2" value="2"/>
-<clearance class="3" value="2"/>
+<clearance class="2" value="1.7"/>
+<clearance class="3" value="1.7"/>
 <clearance class="4" value="1.5"/>
 </class>
@@
 <attribute name="LCSC_PART" value="C25091"/>
 </part>
-<part name="C18" library="BSB-LAN" deviceset="CPOL-EU" device="SMCD" value="220uF 25V">
-<attribute name="LCSC_PART" value=""/>
-</part>
-<part name="C20" library="BSB-LAN" deviceset="C-EU" device="C1808" value="1nF 3kV">
-<attribute name="LCSC_PART" value="C577300"/>
-</part>
-<part name="C21" library="BSB-LAN" deviceset="C-EU" device="C1808" value="1nF 3kV">
-<attribute name="LCSC_PART" value="C577300"/>
+<part name="C18" library="BSB-LAN" deviceset="CPOL-EU" device="SMCD" value="100uF 20V">
+<attribute name="LCSC_PART" value="C7224"/>
+</part>
+<part name="C20" library="BSB-LAN" deviceset="C-EU" device="C1206L" value="1nF 2kV">
+<attribute name="LCSC_PART" value="C9196"/>
+</part>
+<part name="C21" library="BSB-LAN" deviceset="C-EU" device="C1206L" value="1nF 2kV">
+<attribute name="LCSC_PART" value="C9196"/>
 </part>
 <part name="C22" library="BSB-LAN" deviceset="C-EU" device="C0805" value="22uF">
 <attribute name="LCSC_PART" value="C45783"/>
 </part>
-<part name="R41" library="BSB-LAN" deviceset="R-EU_" device="R0402" value="12.1k 1%">
-<attribute name="LCSC_PART" value="C25852"/>
-</part>
-<part name="R40" library="BSB-LAN" deviceset="R-EU_" device="R0402" value="180k 1%">
-<attribute name="LCSC_PART" value="C25760"/>
-</part>
-<part name="R42" library="BSB-LAN" deviceset="R-EU_" device="R0402" value="28.7k 1%">
-<attribute name="LCSC_PART" value="C26972"/>
+<part name="R41" library="BSB-LAN" deviceset="R-EU_" device="R0402" value="22k 1%">
+<attribute name="LCSC_PART" value="C25768"/>
+</part>
+<part name="R40" library="BSB-LAN" deviceset="R-EU_" device="R0402" value="200k 1%">
+<attribute name="LCSC_PART" value="C25764"/>
+</part>
+<part name="R42" library="BSB-LAN" deviceset="R-EU_" device="R0402" value="22k 1%">
+<attribute name="LCSC_PART" value="C25768"/>
 </part>
 <part name="L4" library="BSB-LAN" deviceset="L-US" device="L4040P" value="2.2uH 1.5A">
@@
 <attribute name="LCSC_PART" value="C45783"/>
 </part>
-<part name="R43" library="BSB-LAN" deviceset="R-EU_" device="R0402" value="180k 1%">
-<attribute name="LCSC_PART" value="C25760"/>
+<part name="R43" library="BSB-LAN" deviceset="R-EU_" device="R0402" value="200k 1%">
+<attribute name="LCSC_PART" value="C25764"/>
 </part>
 <part name="R44" library="BSB-LAN" deviceset="R-EU_" device="R0603L" value="330k">
@@
 </part>
 <part name="Q7" library="BSB-LAN" deviceset="WPM2015" device="" technology="-3/TR"/>
-<part name="D6" library="BSB-LAN" deviceset="DIODE-" device="SMB" value="SS510B">
-<attribute name="LCSC_PART" value="C65011"/>
+<part name="D6" library="BSB-LAN" deviceset="DIODE-" device="SMA" value="SS34">
+<attribute name="LCSC_PART" value="C8678"/>
 </part>
 <part name="R47" library="BSB-LAN" deviceset="R-EU_" device="R0402" value="10k">
@@
 Isolated DC
 Supply Iface</text>
-<text x="111.76" y="43.18" size="1.4224" layer="97" font="vector" ratio="10" align="center-left">Vout = 0.6 x (180/40.8 + 1) = 3.25V</text>
+<text x="111.76" y="43.18" size="1.4224" layer="97" font="vector" ratio="10" align="center-left">Vout = 0.6 x (200/44 + 1) = 3.32V</text>
 </plain>
 <instances>

Commit message: Correct ESP32 Prog Control + Update Libraries
1. Correct the control of automatic bootloader entry by adding missing resistor from GPIO2 to GPIO0.
2. Update libraries and fix layout to account for changes.
3. Change the LAN versions of the boards to use the ESP32 with external antenna. If the PCB antenna is used then it is not possible to get the PCB into the enclosure because components stick out on both ends!
Parts:
- added R51: 220R, BSB-LAN:R-EU_R0402
Connections:
- net ESP-GPIO0: now also R51.1
- net ESP-SD-DATA: now also R51.2
Changed lines of the file:
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@@
 <schematic xreflabel="%F%N/%S.%C%R" xrefpart="/%S.%C%R">
 <attributes>
-<attribute name="REVISION" value="v1.0"/>
+<attribute name="REVISION" value="v1.1"/>
 </attributes>
 <variantdefs>
@@
 <attribute name="LCSC_PART" value="C148213"/>
 </part>
+<part name="R51" library="BSB-LAN" deviceset="R-EU_" device="R0402" value="220R">
+<attribute name="LCSC_PART" value="C25091"/>
+</part>
 </parts>
 <sheets>
@@
 <instance part="RN4" gate="G$1" x="55.88" y="43.18" rot="MR90">
 <attribute name="LCSC_PART" x="55.88" y="43.18" size="1.4224" layer="96" font="vector" ratio="10" rot="MR90" align="center" display="off"/>
+</instance>
+<instance part="R51" gate="G$1" x="104.14" y="48.26" rot="MR0">
+<attribute name="LCSC_PART" x="104.14" y="48.26" size="1.4224" layer="96" font="vector" ratio="10" align="center" display="off"/>
 </instance>
 </instances>
@@
 <junction x="187.96" y="121.92"/>
 </segment>
+<segment>
+<wire x1="99.06" y1="48.26" x2="96.52" y2="48.26" width="0.1524" layer="91"/>
+<label x="96.52" y="48.26" size="1.4224" layer="95" font="vector" ratio="10" rot="MR0" xref="yes"/>
+<pinref part="R51" gate="G$1" pin="2"/>
+</segment>
 </net>
 <net name="ESP-SD-CLK" class="4">
@@
 <net name="ESP-GPIO0" class="4">
 <segment>
-<wire x1="116.84" y1="53.34" x2="114.3" y2="53.34" width="0.1524" layer="91"/>
-<label x="114.3" y="53.34" size="1.4224" layer="95" font="vector" ratio="10" rot="R180" xref="yes"/>
+<wire x1="116.84" y1="53.34" x2="111.76" y2="53.34" width="0.1524" layer="91"/>
+<label x="96.52" y="53.34" size="1.4224" layer="95" font="vector" ratio="10" rot="R180" xref="yes"/>
 <pinref part="Q5" gate="G$1" pin="C"/>
+<wire x1="111.76" y1="53.34" x2="96.52" y2="53.34" width="0.1524" layer="91"/>
 <wire x1="116.84" y1="50.8" x2="116.84" y2="53.34" width="0.1524" layer="91"/>
+<pinref part="R51" gate="G$1" pin="1"/>
+<wire x1="109.22" y1="48.26" x2="111.76" y2="48.26" width="0.1524" layer="91"/>
+<wire x1="111.76" y1="48.26" x2="111.76" y2="53.34" width="0.1524" layer="91"/>
+<junction x="111.76" y="53.34"/>
 </segment>
 <segment>
@@
 </segment>
 <segment>
-<wire x1="157.48" y1="58.42" x2="114.3" y2="58.42" width="0.1524" layer="91"/>
-<label x="114.3" y="58.42" size="1.4224" layer="95" font="vector" ratio="10" rot="MR0" xref="yes"/>
+<wire x1="157.48" y1="58.42" x2="96.52" y2="58.42" width="0.1524" layer="91"/>
+<label x="96.52" y="58.42" size="1.4224" layer="95" font="vector" ratio="10" rot="MR0" xref="yes"/>
 <pinref part="IC6" gate="G$1" pin="RXD"/>
 </segment>
@@
 </segment>
 <segment>
-<wire x1="124.46" y1="63.5" x2="114.3" y2="63.5" width="0.1524" layer="91"/>
-<label x="114.3" y="63.5" size="1.4224" layer="95" font="vector" ratio="10" rot="MR0" xref="yes"/>
+<wire x1="124.46" y1="63.5" x2="96.52" y2="63.5" width="0.1524" layer="91"/>
+<label x="96.52" y="63.5" size="1.4224" layer="95" font="vector" ratio="10" rot="MR0" xref="yes"/>
 <pinref part="R49" gate="G$1" pin="2"/>
 </segment>
