File: BSB-to-PoELAN.sch (EAGLE design)
At the start: 121 parts, among them IC1 LAN8710A-EZC, IC2 TPS2376DDA, IC3 TX4138, IC4 SY8089AAAC, IC6 CH340X, Q1 BC847, Q2 BC857, Q3 BC847, Q4 WPM2015-3/TR, Q5 BC847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

Commit message: Add BSB Tx Enable Control
Move the UEXT RX on GPIO35 (input only), and use GPIO32 instead for controlling whether the BSB-TXD pin can drive the optocoupler. This basically replaces the +3.3V connection on the emitter of the invert transistor.

What this means is that when the ESP32 has not yet booted, or if it crashes along the way, the BSB bus is not being driven into TX mode by the pull-down bootstrap resistor. This should stop BSB bus short detection errors when the unit is powered off or has not yet started up.

This will require custom code in the BSB firmware setup (BSB_LAN_custom_setup.h) to configure the enable pin to be an output and driven high. Until that is done the BSB bus remains passive.
Parts:
- added R52: 4.7k, BSB-LAN:R-EU_R0402
Connections:
- new net BSB-ENB: ESP1.GPIO32, Q2.E, R52.2
- net +3.3V: no longer Q2.E
- net GND: now also R52.1
- net UEXT-RX: now also ESP1.GPIO35; no longer ESP1.GPIO32
Changed lines of the file:
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@@
 <attribute name="LCSC_PART" value="C25744"/>
 </part>
-<part name="R8" library="BSB-LAN" deviceset="R-EU_" device="R0402" value="4.7k">
+<part name="R52" library="BSB-LAN" deviceset="R-EU_" device="R0402" value="4.7k">
 <attribute name="LCSC_PART" value="C25900"/>
 </part>
@@
 <part name="R51" library="BSB-LAN" deviceset="R-EU_" device="R0402" value="220R">
 <attribute name="LCSC_PART" value="C25091"/>
+</part>
+<part name="R8" library="BSB-LAN" deviceset="R-EU_" device="R0402" value="4.7k">
+<attribute name="LCSC_PART" value="C25900"/>
 </part>
 </parts>
@@
 <junction x="66.04" y="20.32"/>
 </segment>
+<segment>
+<wire x1="76.2" y1="88.9" x2="83.82" y2="88.9" width="0.1524" layer="91"/>
+<label x="83.82" y="88.9" size="1.4224" layer="95" font="vector" ratio="10" xref="yes"/>
+<pinref part="ESP1" gate="G$1" pin="GPIO35"/>
+</segment>
+</net>
+<net name="BSB-ENB" class="0">
 <segment>
 <wire x1="76.2" y1="96.52" x2="83.82" y2="96.52" width="0.1524" layer="91"/>
@@
 </instance>
 <instance part="U$3" gate="G$1" x="241.3" y="35.56"/>
+<instance part="R52" gate="G$1" x="195.58" y="137.16" rot="R90">
+<attribute name="LCSC_PART" x="195.58" y="137.16" size="2.54" layer="96" font="vector" ratio="10" rot="R90" align="center" display="off"/>
+</instance>
 <instance part="R8" gate="G$1" x="187.96" y="137.16" rot="R90">
 <attribute name="LCSC_PART" x="187.96" y="137.16" size="2.54" layer="96" font="vector" ratio="10" rot="R90" align="center" display="off"/>
@@
 <pinref part="OK2" gate="G$1" pin="C"/>
 <wire x1="152.4" y1="129.54" x2="187.96" y2="129.54" width="0.1524" layer="91"/>
-<label x="190.5" y="129.54" size="1.4224" layer="95" font="vector" ratio="10" xref="yes"/>
+<label x="200.66" y="129.54" size="1.4224" layer="95" font="vector" ratio="10" xref="yes"/>
+<pinref part="R52" gate="G$1" pin="1"/>
+<wire x1="187.96" y1="129.54" x2="195.58" y2="129.54" width="0.1524" layer="91"/>
+<wire x1="195.58" y1="129.54" x2="200.66" y2="129.54" width="0.1524" layer="91"/>
+<wire x1="195.58" y1="132.08" x2="195.58" y2="129.54" width="0.1524" layer="91"/>
+<junction x="195.58" y="129.54"/>
 <pinref part="R8" gate="G$1" pin="1"/>
-<wire x1="187.96" y1="129.54" x2="190.5" y2="129.54" width="0.1524" layer="91"/>
 <wire x1="187.96" y1="132.08" x2="187.96" y2="129.54" width="0.1524" layer="91"/>
 <junction x="187.96" y="129.54"/>
@@
 </net>
 <net name="+3.3V" class="4">
-<segment>
-<pinref part="Q2" gate="G$1" pin="E"/>
-<wire x1="167.64" y1="149.86" x2="167.64" y2="157.48" width="0.1524" layer="91"/>
-<wire x1="167.64" y1="157.48" x2="190.5" y2="157.48" width="0.1524" layer="91"/>
-<label x="190.5" y="157.48" size="1.4224" layer="95" font="vector" ratio="10" xref="yes"/>
-</segment>
 <segment>
 <pinref part="OK1" gate="G$1" pin="COL"/>
@@
 <net name="BSB-TXD" class="4">
 <segment>
-<label x="190.5" y="144.78" size="1.4224" layer="95" font="vector" ratio="10" xref="yes"/>
+<label x="200.66" y="144.78" size="1.4224" layer="95" font="vector" ratio="10" xref="yes"/>
 <pinref part="R6" gate="G$1" pin="2"/>
 <wire x1="185.42" y1="144.78" x2="187.96" y2="144.78" width="0.1524" layer="91"/>
 <pinref part="R8" gate="G$1" pin="2"/>
-<wire x1="187.96" y1="144.78" x2="190.5" y2="144.78" width="0.1524" layer="91"/>
-<wire x1="187.96" y1="142.24" x2="187.96" y2="144.78" width="0.1524" layer="91"/>
+<wire x1="187.96" y1="144.78" x2="200.66" y2="144.78" width="0.1524" layer="91"/>
+<wire x1="187.96" y1="144.78" x2="187.96" y2="142.24" width="0.1524" layer="91"/>
 <junction x="187.96" y="144.78"/>
 </segment>
@@
 </segment>
 </net>
+<net name="BSB-ENB" class="0">
+<segment>
+<pinref part="Q2" gate="G$1" pin="E"/>
+<wire x1="167.64" y1="149.86" x2="167.64" y2="157.48" width="0.1524" layer="91"/>
+<wire x1="167.64" y1="157.48" x2="195.58" y2="157.48" width="0.1524" layer="91"/>
+<label x="200.66" y="157.48" size="1.4224" layer="95" font="vector" ratio="10" xref="yes"/>
+<pinref part="R52" gate="G$1" pin="2"/>
+<wire x1="195.58" y1="157.48" x2="200.66" y2="157.48" width="0.1524" layer="91"/>
+<wire x1="195.58" y1="142.24" x2="195.58" y2="157.48" width="0.1524" layer="91"/>
+<junction x="195.58" y="157.48"/>
+</segment>
+</net>
