File: BSB-to-Wifi.brd (EAGLE design)
At the start: 86.5 x 32.8 mm, 73 parts, among them IC4 SY8089AAAC, IC6 CH340X, Q1 BC847, Q2 BC857, Q5 BC847, Q6 BC847, Q7 WPM2015-3/TR, U2 ESDS314DBV

Commit message: Add BSB Tx Enable Control
Move the UEXT RX on GPIO35 (input only), and use GPIO32 instead for controlling whether the BSB-TXD pin can drive the optocoupler. This basically replaces the +3.3V connection on the emitter of the invert transistor.

What this means is that when the ESP32 has not yet booted, or if it crashes along the way, the BSB bus is not being driven into TX mode by the pull-down bootstrap resistor. This should stop BSB bus short detection errors when the unit is powered off or has not yet started up.

This will require custom code in the BSB firmware setup (BSB_LAN_custom_setup.h) to configure the enable pin to be an output and driven high. Until that is done the BSB bus remains passive.
Parts:
- added R11: 4.7k, BSB-LAN:R0402
Connections:
- new net BSB-ENB: ESP1.8, Q2.E, R11.2
- net +3.3V: no longer Q2.E
- net GND: now also R11.1
- net UEXT-RX: now also ESP1.7; no longer ESP1.8
Routing:
- net BSB-ENB: track 0.00 -> 50.0 mm, vias 0 -> 2
- net +3.3V: track 26.3 -> 24.3 mm
- net UEXT-RX: track 45.3 -> 46.7 mm
- net BSB-TXD: track 51.6 -> 52.1 mm
